Commit message: updates to material name in urdf to comply with isaacsim standards, added small box to virtual joint. Both of these remove a large number of warnings in the terminal.

File: source/ryan_tasks/ryan_tasks/tasks/robots/so101_new_calib.urdf (robot description, URDF)
Before this commit: robot so101_new_calib, 8 links, 7 joints
Links:
- link gripper_frame_link: geometry visual box size=0.001 0.001 0.001
Joints:
- joint gripper_frame_joint: axis 0 0 0 -> (none)

Commit message: Updated reach task with my current configuration. Learns signficantly better, paired with the updates to the ppo implementation. Also updated the urdf to more closely match my robot, and joint ranges to match my robot. My robot had slightly more range of motion on most joints than the urdf defined.

File: source/ryan_tasks/ryan_tasks/tasks/robots/so101_new_calib.urdf (robot description, URDF)
Before this commit: robot so101_new_calib, 8 links, 7 joints
Joints:
- joint elbow_flex: limit lower=-1.69 upper=1.69 effort=10 velocity=10 -> lower=-1.69582 upper=1.69582 effort=10 velocity=10
- joint shoulder_lift: limit lower=-1.74533 upper=1.74533 effort=10 velocity=10 -> lower=-1.85151 upper=1.85151 effort=10 velocity=10
- joint shoulder_pan: limit lower=-1.91986 upper=1.91986 effort=10 velocity=10 -> lower=-2.07164 upper=2.07164 effort=10 velocity=10
- joint wrist_flex: limit lower=-1.65806 upper=1.65806 effort=10 velocity=10 -> lower=-1.84329 upper=1.75850 effort=10 velocity=10
- joint wrist_roll: limit lower=-2.74385 upper=2.84121 effort=10 velocity=10 -> lower=-3.08586 upper=3.19579 effort=10 velocity=10
